File: gameblaster.kicad_sch (KiCad schematic)
At the start: 74 parts, among them IC1 TEA2025, IC11 74LS08, IC12 74LS74, IC2 SAA1099, IC3 SAA1099, IC4 74LS245, IC5 74LS374, IC6 74LS138, IC7 74LS138, IC8 74LS32, IC9 74LS125, J1 Conn_02x06_Odd_Even

Commit message: update pdf
Parts:
- renumbered IC9 to IC10, IC11 to IC9
Changed lines of the file:
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@@
   (symbol (lib_id "74xx:74LS08") (at 260.985 125.095 0) (unit 4)
     (in_bom yes) (on_board yes) (fields_autoplaced)
-    (property "Reference" "IC11" (id 0) (at 260.985 117.5852 0))
+    (property "Reference" "IC9" (id 0) (at 260.985 117.5852 0))
     (property "Value" "74LS08" (id 1) (at 260.985 120.1221 0))
     (property "Footprint" "gameblaster:DIP254P762X635-14" (id 2) (at 260.985 125.095 0)
@@
   (symbol (lib_id "74xx:74LS08") (at 287.02 258.445 0) (unit 3)
     (in_bom yes) (on_board yes) (fields_autoplaced)
-    (property "Reference" "IC11" (id 0) (at 287.02 250.9352 0))
+    (property "Reference" "IC9" (id 0) (at 287.02 250.9352 0))
     (property "Value" "74LS08" (id 1) (at 287.02 253.4721 0))
     (property "Footprint" "gameblaster:DIP254P762X635-14" (id 2) (at 287.02 258.445 0)
@@
   (symbol (lib_id "74xx:74LS125") (at 311.785 113.665 0) (unit 3)
     (in_bom yes) (on_board yes) (fields_autoplaced)
-    (property "Reference" "IC9" (id 0) (at 311.785 106.1552 0))
+    (property "Reference" "IC10" (id 0) (at 311.785 106.1552 0))
     (property "Value" "74LS125" (id 1) (at 311.785 108.6921 0))
     (property "Footprint" "gameblaster:DIP254P762X635-14" (id 2) (at 311.785 113.665 0)
@@
   (symbol (lib_id "74xx:74LS08") (at 387.35 133.985 90) (unit 5)
     (in_bom yes) (on_board yes) (fields_autoplaced)
-    (property "Reference" "IC11" (id 0) (at 387.35 125.2052 90))
+    (property "Reference" "IC9" (id 0) (at 387.35 125.2052 90))
     (property "Value" "74LS08" (id 1) (at 387.35 127.7421 90))
     (property "Footprint" "gameblaster:DIP254P762X635-14" (id 2) (at 387.35 133.985 0)
@@
   (symbol (lib_id "74xx:74LS125") (at 245.745 274.955 0) (unit 4)
     (in_bom yes) (on_board yes) (fields_autoplaced)
-    (property "Reference" "IC9" (id 0) (at 245.745 267.4452 0))
+    (property "Reference" "IC10" (id 0) (at 245.745 267.4452 0))
     (property "Value" "74LS125" (id 1) (at 245.745 269.9821 0))
     (property "Footprint" "gameblaster:DIP254P762X635-14" (id 2) (at 245.745 274.955 0)
@@
   (symbol (lib_id "74xx:74LS125") (at 387.35 112.395 90) (unit 5)
     (in_bom yes) (on_board yes) (fields_autoplaced)
-    (property "Reference" "IC9" (id 0) (at 387.35 103.6152 90))
+    (property "Reference" "IC10" (id 0) (at 387.35 103.6152 90))
     (property "Value" "74LS125" (id 1) (at 387.35 106.1521 90))
     (property "Footprint" "gameblaster:DIP254P762X635-14" (id 2) (at 387.35 112.395 0)
@@
   (symbol (lib_id "74xx:74LS08") (at 146.05 111.76 0) (unit 1)
     (in_bom yes) (on_board yes) (fields_autoplaced)
-    (property "Reference" "IC11" (id 0) (at 146.05 104.2502 0))
+    (property "Reference" "IC9" (id 0) (at 146.05 104.2502 0))
     (property "Value" "74LS08" (id 1) (at 146.05 106.7871 0))
     (property "Footprint" "gameblaster:DIP254P762X635-14" (id 2) (at 146.05 111.76 0)
@@
   (symbol (lib_id "74xx:74LS125") (at 260.985 104.775 0) (unit 2)
     (in_bom yes) (on_board yes) (fields_autoplaced)
-    (property "Reference" "IC9" (id 0) (at 260.985 97.2652 0))
+    (property "Reference" "IC10" (id 0) (at 260.985 97.2652 0))
     (property "Value" "74LS125" (id 1) (at 260.985 99.8021 0))
     (property "Footprint" "gameblaster:DIP254P762X635-14" (id 2) (at 260.985 104.775 0)
@@
   (symbol (lib_id "74xx:74LS125") (at 260.985 139.065 0) (unit 1)
     (in_bom yes) (on_board yes) (fields_autoplaced)
-    (property "Reference" "IC9" (id 0) (at 260.985 131.5552 0))
+    (property "Reference" "IC10" (id 0) (at 260.985 131.5552 0))
     (property "Value" "74LS125" (id 1) (at 260.985 134.0921 0))
     (property "Footprint" "gameblaster:DIP254P762X635-14" (id 2) (at 260.985 139.065 0)
@@
   (symbol (lib_id "74xx:74LS08") (at 267.97 258.445 0) (unit 2)
     (in_bom yes) (on_board yes) (fields_autoplaced)
-    (property "Reference" "IC11" (id 0) (at 267.97 250.9352 0))
+    (property "Reference" "IC9" (id 0) (at 267.97 250.9352 0))
     (property "Value" "74LS08" (id 1) (at 267.97 253.4721 0))
     (property "Footprint" "gameblaster:DIP254P762X635-14" (id 2) (at 267.97 258.445 0)
@@
       (reference "IC8") (unit 5) (value "74LS32") (footprint "gameblaster:DIP254P762X635-14")
     )
+    (path "/765545db-fdf8-4088-b879-4ed9d866d54c"
+      (reference "IC9") (unit 1) (value "74LS08") (footprint "gameblaster:DIP254P762X635-14")
+    )
+    (path "/e803b058-2edc-400e-9688-6577a8c7ba67"
+      (reference "IC9") (unit 2) (value "74LS08") (footprint "gameblaster:DIP254P762X635-14")
+    )
+    (path "/0b57a4b6-1948-4aca-b637-464401fa822e"
+      (reference "IC9") (unit 3) (value "74LS08") (footprint "gameblaster:DIP254P762X635-14")
+    )
+    (path "/09dc38b1-1021-4ac6-a2dc-fa43c803f232"
+      (reference "IC9") (unit 4) (value "74LS08") (footprint "gameblaster:DIP254P762X635-14")
+    )
+    (path "/40931a71-11a3-4fe8-94c8-f868e40a53de"
+      (reference "IC9") (unit 5) (value "74LS08") (footprint "gameblaster:DIP254P762X635-14")
+    )
     (path "/c4a3e094-0752-4c25-948c-f70b9f50db69"
-      (reference "IC9") (unit 1) (value "74LS125") (footprint "gameblaster:DIP254P762X635-14")
+      (reference "IC10") (unit 1) (value "74LS125") (footprint "gameblaster:DIP254P762X635-14")
     )
     (path "/831292c1-c891-455c-896d-2aa430beaa1e"
-      (reference "IC9") (unit 2) (value "74LS125") (footprint "gameblaster:DIP254P762X635-14")
+      (reference "IC10") (unit 2) (value "74LS125") (footprint "gameblaster:DIP254P762X635-14")
     )
     (path "/35c6d805-db92-42ea-8156-ac58fe604c23"
-      (reference "IC9") (unit 3) (value "74LS125") (footprint "gameblaster:DIP254P762X635-14")
+      (reference "IC10") (unit 3) (value "74LS125") (footprint "gameblaster:DIP254P762X635-14")
     )
     (path "/5f06f0b0-bd31-4b6f-bf5a-59c87a3b785d"
-      (reference "IC9") (unit 4) (value "74LS125") (footprint "gameblaster:DIP254P762X635-14")
+      (reference "IC10") (unit 4) (value "74LS125") (footprint "gameblaster:DIP254P762X635-14")
     )
     (path "/72697600-3dd6-49ff-81ec-b4ba443a8d83"
-      (reference "IC9") (unit 5) (value "74LS125") (footprint "gameblaster:DIP254P762X635-14")
-    )
-    (path "/765545db-fdf8-4088-b879-4ed9d866d54c"
-      (reference "IC11") (unit 1) (value "74LS08") (footprint "gameblaster:DIP254P762X635-14")
-    )
-    (path "/e803b058-2edc-400e-9688-6577a8c7ba67"
-      (reference "IC11") (unit 2) (value "74LS08") (footprint "gameblaster:DIP254P762X635-14")
-    )
-    (path "/0b57a4b6-1948-4aca-b637-464401fa822e"
-      (reference "IC11") (unit 3) (value "74LS08") (footprint "gameblaster:DIP254P762X635-14")
-    )
-    (path "/09dc38b1-1021-4ac6-a2dc-fa43c803f232"
-      (reference "IC11") (unit 4) (value "74LS08") (footprint "gameblaster:DIP254P762X635-14")
-    )
-    (path "/40931a71-11a3-4fe8-94c8-f868e40a53de"
-      (reference "IC11") (unit 5) (value "74LS08") (footprint "gameblaster:DIP254P762X635-14")
+      (reference "IC10") (unit 5) (value "74LS125") (footprint "gameblaster:DIP254P762X635-14")
     )
     (path "/00000000-0000-0000-0000-000063dc9675"
